Commit message: Add base_footprint

File: factomove_description/urdf/factomove_core.xacro (robot description, xacro)
@@ -1,10 +1,10 @@
 <?xml version="1.0"?>
 <robot xmlns:xacro="http://www.ros.org/wiki/xacro">
-    <!-- <link name="base_footprint"/>
+    <link name="base_footprint"/>
   <joint name="base_joint" type="fixed">
     <parent link="base_footprint"/>
     <child link="base_link" />
-    <origin xyz="0 0 0.010" rpy="0 0 0"/>
-  </joint> -->
+    <origin xyz="0 0 0.21" rpy="0 0 0"/>
+  </joint>
     <!-- ============= BASE LINK ============= -->
     <link name="base_link">
