Commit message: Add simulation

File: factomove_description/urdf/factomove.urdf.xacro (robot description, xacro)
@@ -2,3 +2,4 @@
 <robot xmlns:xacro="http://www.ros.org/wiki/xacro"  name="factomove">
     <xacro:include filename="factomove_core.xacro" />
+    <xacro:include filename="factomove.gazebo" />
 </robot>

File: factomove_description/urdf/factomove_core.xacro (robot description, xacro)
@@ -2,9 +2,9 @@
 <robot xmlns:xacro="http://www.ros.org/wiki/xacro">
     <link name="base_footprint"/>
-  <joint name="base_joint" type="fixed">
-    <parent link="base_footprint"/>
-    <child link="base_link" />
-    <origin xyz="0 0 0.21" rpy="0 0 0"/>
-  </joint>
+    <joint name="base_joint" type="fixed">
+        <parent link="base_footprint"/>
+        <child link="base_link" />
+        <origin xyz="0 0 0.21" rpy="0 0 0"/>
+    </joint>
     <!-- ============= BASE LINK ============= -->
     <link name="base_link">
@@ -53,5 +53,5 @@
         </collision>
     </link>
-    <joint name="left_wheel" type="continuous">
+    <joint name="left_wheel_joint" type="continuous">
         <origin xyz="0 0.224 -0.141" rpy="0 0 0" />
         <parent link="base_link" />
@@ -84,5 +84,5 @@
         </collision>
     </link>
-    <joint name="right_wheel" type="continuous">
+    <joint name="right_wheel_joint" type="continuous">
         <origin xyz="0 -0.224 -0.141" rpy="0 0 0" />
         <parent link="base_link" />

Commit message: Add move in simulation

File: factomove_description/urdf/factomove.urdf.xacro (robot description, xacro)
@@ -2,4 +2,4 @@
 <robot xmlns:xacro="http://www.ros.org/wiki/xacro"  name="factomove">
     <xacro:include filename="factomove_core.xacro" />
-    <!-- <xacro:include filename="factomove.gazebo" /> -->
+    <xacro:include filename="factomove.gazebo" />
 </robot>

File: factomove_description/urdf/factomove_core.xacro (robot description, xacro)
@@ -1,9 +1,9 @@
 <?xml version="1.0"?>
 <robot xmlns:xacro="http://www.ros.org/wiki/xacro">
-    <link name="base_footprint"/>
+    <link name="base_footprint"> </link>
     <joint name="base_joint" type="fixed">
-        <parent link="base_footprint"/>
+        <parent link="base_footprint" />
         <child link="base_link" />
-        <origin xyz="0 0 0.21" rpy="0 0 0"/>
+        <origin xyz="0 0 0.21" rpy="0 0 0" />
     </joint>
     <!-- ============= BASE LINK ============= -->
@@ -12,5 +12,6 @@
             <origin xyz="6.1085E-11 7.0637E-11 -0.058359" rpy="0 0 0" />
             <mass value="11.93" />
-            <inertia ixx="0.24655" ixy="1.0146E-10" ixz="-7.2198E-14" iyy="0.44294" iyz="1.8415E-13" izz="0.61972" />
+            <inertia ixx="0.24655" ixy="1.0146E-10" ixz="-7.2198E-14" iyy="0.44294" iyz="1.8415E-13"
+                izz="0.61972" />
         </inertial>
         <visual>
@@ -35,5 +36,6 @@
             <origin xyz="-6.3781E-06 -0.027802 1.0717E-06" rpy="0 0 0" />
             <mass value="1.0785" />
-            <inertia ixx="0.0019839" ixy="-3.8726E-07" ixz="-5.7089E-09" iyy="0.0033904" iyz="6.5067E-08" izz="0.0019839" />
+            <inertia ixx="0.0019839" ixy="-3.8726E-07" ixz="-5.7089E-09" iyy="0.0033904"
+                iyz="6.5067E-08" izz="0.0019839" />
         </inertial>
         <visual>
@@ -43,6 +45,6 @@
             </geometry>
             <material name="">
-                    <color rgba="0.79216 0.81961 0.93333 1" />
-                </material>
+                <color rgba="0.79216 0.81961 0.93333 1" />
+            </material>
         </visual>
         <collision>
@@ -58,6 +60,6 @@
         <child link="left_wheel" />
         <axis xyz="0 1 0" />
-        <limit effort="10" velocity="10" />
-        <dynamics damping="0.1" friction="0.1" />
+        <limit effort="50000" velocity="10" />
+        <dynamics damping="1.0" friction="1.0" />
     </joint>
     <!-- ============= RIGHT WHEEL ============= -->
@@ -66,5 +68,6 @@
             <origin xyz="3.043E-06 0.027802 -5.7069E-06" rpy="0 0 0" />
             <mass value="1.0785" />
-            <inertia ixx="0.0019839" ixy="-1.8476E-07" ixz="-1.4505E-08" iyy="0.0033904" iyz="3.465E-07" izz="0.0019839" />
+            <inertia ixx="0.0019839" ixy="-1.8476E-07" ixz="-1.4505E-08" iyy="0.0033904"
+                iyz="3.465E-07" izz="0.0019839" />
         </inertial>
         <visual>
@@ -89,6 +92,6 @@
         <child link="right_wheel" />
         <axis xyz="0 1 0" />
-        <limit effort="10" velocity="10" />
-        <dynamics damping="0.1" friction="0.1" />
+        <limit effort="50000" velocity="10" />
+        <dynamics damping="1.0" friction="1.0" />
     </joint>
     <!-- ============= FRONT LEFT KEEPER ============= -->
@@ -134,5 +137,6 @@
             <origin xyz="-3.8734E-09 1.1658E-09 3.0966E-09" rpy="0 0 0" />
             <mass value="0.67052" />
-            <inertia ixx="0.0015386" ixy="4.1231E-06" ixz="-5.9599E-12" iyy="0.0028064" iyz="2.5984E-12" izz="0.0015386" />
+            <inertia ixx="0.0015386" ixy="4.1231E-06" ixz="-5.9599E-12" iyy="0.0028064"
+                iyz="2.5984E-12" izz="0.0015386" />
         </inertial>
         <visual>
@@ -165,5 +169,6 @@
             <origin xyz="-0.026628 0.00066635 -0.039345" rpy="0 0 0" />
             <mass value="0.10281" />
-            <inertia ixx="0.00019502" ixy="-1.2185E-07" ixz="-4.081E-05" iyy="0.00016739" iyz="9.2462E-08" izz="0.00019502" />
+            <inertia ixx="0.00019502" ixy="-1.2185E-07" ixz="-4.081E-05" iyy="0.00016739"
+                iyz="9.2462E-08" izz="0.00019502" />
         </inertial>
         <visual>
@@ -196,5 +201,6 @@
             <origin xyz="-3.8734E-09 1.1658E-09 3.0966E-09" rpy="0 0 0" />
             <mass value="0.67052" />
-            <inertia ixx="0.0015386" ixy="4.1231E-06" ixz="-5.9599E-12" iyy="0.0028064" iyz="2.5984E-12" izz="0.0015386" />
+            <inertia ixx="0.0015386" ixy="4.1231E-06" ixz="-5.9599E-12" iyy="0.0028064"
+                iyz="2.5984E-12" izz="0.0015386" />
         </inertial>
         <visual>
@@ -227,5 +233,6 @@
             <origin xyz="-0.026628 0.00066635 -0.039345" rpy="0 0 0" />
             <mass value="0.10281" />
-            <inertia ixx="0.00019502" ixy="-1.2185E-07" ixz="-4.081E-05" iyy="0.00016739" iyz="9.2462E-08" izz="0.00019502" />
+            <inertia ixx="0.00019502" ixy="-1.2185E-07" ixz="-4.081E-05" iyy="0.00016739"
+                iyz="9.2462E-08" izz="0.00019502" />
         </inertial>
         <visual>
@@ -258,5 +265,6 @@
             <origin xyz="-3.8734E-09 1.1658E-09 3.0966E-09" rpy="0 0 0" />
             <mass value="0.67052" />
-            <inertia ixx="0.0015386" ixy="4.1231E-06" ixz="-5.9599E-12" iyy="0.0028064" iyz="2.5984E-12" izz="0.0015386" />
+            <inertia ixx="0.0015386" ixy="4.1231E-06" ixz="-5.9599E-12" iyy="0.0028064"
+                iyz="2.5984E-12" izz="0.0015386" />
         </inertial>
         <visual>
@@ -289,5 +297,6 @@
             <origin xyz="-0.026628 0.00066635 -0.039345" rpy="0 0 0" />
             <mass value="0.10281" />
-            <inertia ixx="0.00019502" ixy="-1.2185E-07" ixz="-4.081E-05" iyy="0.00016739" iyz="9.2462E-08" izz="0.00019502" />
+            <inertia ixx="0.00019502" ixy="-1.2185E-07" ixz="-4.081E-05" iyy="0.00016739"
+                iyz="9.2462E-08" izz="0.00019502" />
         </inertial>
         <visual>
@@ -320,5 +329,6 @@
             <origin xyz="-3.8734E-09 1.1658E-09 3.0966E-09" rpy="0 0 0" />
             <mass value="0.67052" />
-            <inertia ixx="0.0015386" ixy="4.1231E-06" ixz="-5.9599E-12" iyy="0.0028064" iyz="2.5984E-12" izz="0.0015386" />
+            <inertia ixx="0.0015386" ixy="4.1231E-06" ixz="-5.9599E-12" iyy="0.0028064"
+                iyz="2.5984E-12" izz="0.0015386" />
         </inertial>
         <visual>
@@ -346,28 +356,3 @@
         <dynamics damping="0.1" friction="0.1" />
     </joint>
-    <!-- ============= BASE SCAN ============= -->
-    <!-- <link name="base_scan">
-        <visual>
-            <origin xyz="0 0 0" rpy="0 0 0"/>
-            <geometry>
-                <mesh filename="package://factomove_description/meshes/hokuyo.dae"/>
-            </geometry>
-        </visual>
-        <collision>
-            <origin xyz="0.015 0 -0.0065" rpy="0 0 0"/>
-            <geometry>
-                <cylinder length="0.0315" radius="0.055"/>
-            </geometry>
-        </collision>
-        <inertial>
-            <mass value="0.114" />
-            <origin xyz="0 0 0" />
-            <inertia ixx="0.001" ixy="0.0" ixz="0.0" iyy="0.001" iyz="0.0" izz="0.001" />
-        </inertial>
-    </link>
-    <joint name="scan_joint" type="fixed">
-        <parent link="base_link"/>
-        <child link="base_scan"/>
-        <origin xyz="-0.064 0 0.122" rpy="0 0 0"/>
-    </joint> -->
 </robot>
